Commit message: Role 2: Switch to Twist msg to fix Bridge error & Update control logic

File: src/pure_pursuit_controller/urdf/ackermann_car.urdf (robot description, URDF)
Before this commit: robot ackermann_bot, 5 links, 4 joints
Links:
- link base_link: mass 5.0 -> 10.0; geometry collision box size=0.5 0.25 0.1; visual box size=0.5 0.25 0.1
- link front_left_wheel: mass 0.2 -> 1.0; geometry collision cylinder length=0.04 radius=0.06; visual cylinder length=0.04 radius=0.06
- link front_right_wheel: mass 0.2 -> 1.0; geometry collision cylinder length=0.04 radius=0.06; visual cylinder length=0.04 radius=0.06
- link rear_left_wheel: mass 0.2 -> 1.0; geometry collision cylinder length=0.04 radius=0.06; visual cylinder length=0.04 radius=0.06
- link rear_right_wheel: mass 0.2 -> 1.0; geometry collision cylinder length=0.04 radius=0.06; visual cylinder length=0.04 radius=0.06
Joints:
- joint front_left_steer_joint: axis 0 1 0 -> 0 0 1; limit lower=-0.6 upper=0.6 effort=10.0 velocity=1.0 -> lower=-0.8 upper=0.8 effort=500.0 velocity=30.0; origin xyz=0.15 0.175 0 rpy=-1.57 0 0 -> xyz=0.15 0.15 -0.05 rpy=-1.57 0 0
- joint front_right_steer_joint: axis 0 1 0 -> 0 0 1; limit lower=-0.6 upper=0.6 effort=10.0 velocity=1.0 -> lower=-0.8 upper=0.8 effort=500.0 velocity=30.0; origin xyz=0.15 -0.175 0 rpy=-1.57 0 0 -> xyz=0.15 -0.15 -0.05 rpy=-1.57 0 0
- joint rear_left_joint: limit (none) -> effort=500.0 velocity=30.0; origin xyz=-0.15 0.175 0 rpy=-1.57 0 0 -> xyz=-0.15 0.15 -0.05 rpy=-1.57 0 0
- joint rear_right_joint: limit (none) -> effort=500.0 velocity=30.0; origin xyz=-0.15 -0.175 0 rpy=-1.57 0 0 -> xyz=-0.15 -0.15 -0.05 rpy=-1.57 0 0

Commit message: Bao fix attempt 9

File: src/pure_pursuit_controller/urdf/ackermann_car.urdf (robot description, URDF)
Before this commit: robot ackermann_bot, 5 links, 4 joints
Joints:
- joint front_left_steer_joint: axis 0 0 1 -> 0 1 0; origin xyz=0.15 0.15 -0.05 rpy=-1.57 0 0 -> xyz=0.15 0.15 -0.05 rpy=0 0 0
- joint front_right_steer_joint: axis 0 0 1 -> 0 1 0; origin xyz=0.15 -0.15 -0.05 rpy=-1.57 0 0 -> xyz=0.15 -0.15 -0.05 rpy=0 0 0
- joint rear_left_joint: axis 0 0 1 -> 0 1 0; origin xyz=-0.15 0.15 -0.05 rpy=-1.57 0 0 -> xyz=-0.15 0.15 -0.05 rpy=0 0 0
- joint rear_right_joint: axis 0 0 1 -> 0 1 0; origin xyz=-0.15 -0.15 -0.05 rpy=-1.57 0 0 -> xyz=-0.15 -0.15 -0.05 rpy=0 0 0

Commit message: alternative path

File: src/pure_pursuit_controller/urdf/ackermann_car.urdf (robot description, URDF)
Before this commit: robot ackermann_bot, 5 links, 4 joints
Links:
- added link base_footprint
- added link front_left_steer, mass 0.1
- added link front_right_steer, mass 0.1
- link base_link: mass 10.0 -> 5.0; geometry collision box size=0.5 0.3 0.1; visual box size=0.5 0.3 0.1
- link front_left_wheel: geometry collision cylinder length=0.05 radius=0.1; visual cylinder length=0.05 radius=0.1
- link front_right_wheel: geometry collision cylinder length=0.05 radius=0.1; visual cylinder length=0.05 radius=0.1
- link rear_left_wheel: geometry collision cylinder length=0.05 radius=0.1; visual cylinder length=0.05 radius=0.1
- link rear_right_wheel: geometry collision cylinder length=0.05 radius=0.1; visual cylinder length=0.05 radius=0.1
Joints:
- added joint base_joint: type fixed, parent base_link, child base_footprint, origin xyz=0 0 -0.15 rpy=0 0 0
- added joint front_left_wheel_joint: type revolute, parent front_left_steer, child front_left_wheel, origin xyz=0 0 0 rpy=-1.5707 0 0, axis 0 0 1, limit lower=-1e16 upper=1e16 effort=10.0 velocity=20.0
- added joint front_right_wheel_joint: type revolute, parent front_right_steer, child front_right_wheel, origin xyz=0 0 0 rpy=-1.5707 0 0, axis 0 0 1, limit lower=-1e16 upper=1e16 effort=10.0 velocity=20.0
- joint front_left_steer_joint: axis 0 1 0 -> 0 0 1; child front_left_wheel -> front_left_steer; limit lower=-0.8 upper=0.8 effort=500.0 velocity=30.0 -> lower=-0.6 upper=0.6 effort=5.0 velocity=5.0; origin xyz=0.15 0.15 -0.05 rpy=0 0 0 -> xyz=0.15 0.175 -0.05 rpy=0 0 0
- joint front_right_steer_joint: axis 0 1 0 -> 0 0 1; child front_right_wheel -> front_right_steer; limit lower=-0.8 upper=0.8 effort=500.0 velocity=30.0 -> lower=-0.6 upper=0.6 effort=5.0 velocity=5.0; origin xyz=0.15 -0.15 -0.05 rpy=0 0 0 -> xyz=0.15 -0.175 -0.05 rpy=0 0 0
- joint rear_left_joint: axis 0 1 0 -> 0 0 1; limit effort=500.0 velocity=30.0 -> lower=-1e16 upper=1e16 effort=10.0 velocity=20.0; origin xyz=-0.15 0.15 -0.05 rpy=0 0 0 -> xyz=-0.15 0.175 -0.05 rpy=-1.5707 0 0; type continuous -> revolute
- joint rear_right_joint: axis 0 1 0 -> 0 0 1; limit effort=500.0 velocity=30.0 -> lower=-1e16 upper=1e16 effort=10.0 velocity=20.0; origin xyz=-0.15 -0.15 -0.05 rpy=0 0 0 -> xyz=-0.15 -0.175 -0.05 rpy=-1.5707 0 0; type continuous -> revolute
